Commit message: a1 learns good walking gait

File: resources/robots/a1/urdf/a1.urdf (robot description, URDF)
Before this commit: robot a1_description, 23 links, 22 joints
Links:
- link FL_hip: geometry collision cylinder length=0.04 radius=0.046; visual mesh filename=../meshes/hip.dae scale=1 1 1
- link FL_thigh_shoulder: geometry collision cylinder length=0.032 radius=0.041
- link FR_hip: geometry collision cylinder length=0.04 radius=0.046; visual mesh filename=../meshes/hip.dae scale=1 1 1
- link FR_thigh_shoulder: geometry collision cylinder length=0.032 radius=0.041
- link RL_hip: geometry collision cylinder length=0.04 radius=0.046; visual mesh filename=../meshes/hip.dae scale=1 1 1
- link RL_thigh_shoulder: geometry collision cylinder length=0.032 radius=0.041
- link RR_hip: geometry collision cylinder length=0.04 radius=0.046; visual mesh filename=../meshes/hip.dae scale=1 1 1
- link RR_thigh_shoulder: geometry collision cylinder length=0.032 radius=0.041
- link imu_link: geometry collision box size=.001 .001 .001; visual box size=0.001 0.001 0.001
- link trunk: mass 4.713 -> 6.0
Joints:
- joint FL_calf_joint: limit lower=-2.69653369433 upper=-0.916297857297 effort=55 velocity=28.6 -> lower=-2.69653369433 upper=-0.916297857297 effort=33.5 velocity=21
- joint FL_hip_joint: limit lower=-0.802851455917 upper=0.802851455917 effort=20 velocity=52.4 -> lower=-0.802851455917 upper=0.802851455917 effort=33.5 velocity=21; origin xyz=0.183 0.047 0 rpy=0 0 0 -> xyz=0.1805 0.047 0 rpy=0 0 0
- joint FL_thigh_joint: limit lower=-1.0471975512 upper=4.18879020479 effort=55 velocity=28.6 -> lower=-1.0471975512 upper=4.18879020479 effort=33.5 velocity=21; origin xyz=0 0.08505 0 rpy=0 0 0 -> xyz=0 0.0838 0 rpy=0 0 0
- joint FR_calf_joint: limit lower=-2.69653369433 upper=-0.916297857297 effort=55 velocity=28.6 -> lower=-2.69653369433 upper=-0.916297857297 effort=33.5 velocity=21
- joint FR_hip_joint: limit lower=-0.802851455917 upper=0.802851455917 effort=20 velocity=52.4 -> lower=-0.802851455917 upper=0.802851455917 effort=33.5 velocity=21; origin xyz=0.183 -0.047 0 rpy=0 0 0 -> xyz=0.1805 -0.047 0 rpy=0 0 0
- joint FR_thigh_joint: limit lower=-1.0471975512 upper=4.18879020479 effort=55 velocity=28.6 -> lower=-1.0471975512 upper=4.18879020479 effort=33.5 velocity=21; origin xyz=0 -0.08505 0 rpy=0 0 0 -> xyz=0 -0.0838 0 rpy=0 0 0
- joint RL_calf_joint: limit lower=-2.69653369433 upper=-0.916297857297 effort=55 velocity=28.6 -> lower=-2.69653369433 upper=-0.916297857297 effort=33.5 velocity=21
- joint RL_hip_joint: limit lower=-0.802851455917 upper=0.802851455917 effort=20 velocity=52.4 -> lower=-0.802851455917 upper=0.802851455917 effort=33.5 velocity=21; origin xyz=-0.183 0.047 0 rpy=0 0 0 -> xyz=-0.1805 0.047 0 rpy=0 0 0
- joint RL_thigh_joint: limit lower=-1.0471975512 upper=4.18879020479 effort=55 velocity=28.6 -> lower=-1.0471975512 upper=4.18879020479 effort=33.5 velocity=21; origin xyz=0 0.08505 0 rpy=0 0 0 -> xyz=0 0.0838 0 rpy=0 0 0
- joint RR_calf_joint: limit lower=-2.69653369433 upper=-0.916297857297 effort=55 velocity=28.6 -> lower=-2.69653369433 upper=-0.916297857297 effort=33.5 velocity=21
- joint RR_hip_joint: limit lower=-0.802851455917 upper=0.802851455917 effort=20 velocity=52.4 -> lower=-0.802851455917 upper=0.802851455917 effort=33.5 velocity=21; origin xyz=-0.183 -0.047 0 rpy=0 0 0 -> xyz=-0.1805 -0.047 0 rpy=0 0 0
- joint RR_thigh_joint: limit lower=-1.0471975512 upper=4.18879020479 effort=55 velocity=28.6 -> lower=-1.0471975512 upper=4.18879020479 effort=33.5 velocity=21; origin xyz=0 -0.08505 0 rpy=0 0 0 -> xyz=0 -0.0838 0 rpy=0 0 0

Commit message: significant config update. Move all configs to yaml

File: resources/robots/a1/urdf/a1.urdf (robot description, URDF)
Before this commit: robot a1_description, 23 links, 22 joints
Links:
- link imu_link: geometry collision box size=.06 .15 .1; visual box size=0.001 0.001 0.001
- link trunk: mass 6.0 -> 4.713
Joints:
- joint FL_calf_joint: limit lower=-2.69653369433 upper=-0.916297857297 effort=33.5 velocity=21 -> lower=-2.69653369433 upper=-0.916297857297 effort=33.5 velocity=28.6
- joint FL_hip_joint: limit lower=-0.802851455917 upper=0.802851455917 effort=33.5 velocity=21 -> lower=-0.802851455917 upper=0.802851455917 effort=33.5 velocity=52.4; origin xyz=0.1805 0.047 0 rpy=0 0 0 -> xyz=0.183 0.047 0 rpy=0 0 0
- joint FL_thigh_joint: limit lower=-1.0471975512 upper=4.18879020479 effort=33.5 velocity=21 -> lower=-1.0471975512 upper=4.18879020479 effort=33.5 velocity=28.6; origin xyz=0 0.0838 0 rpy=0 0 0 -> xyz=0 0.08505 0 rpy=0 0 0
- joint FR_calf_joint: limit lower=-2.69653369433 upper=-0.916297857297 effort=33.5 velocity=21 -> lower=-2.69653369433 upper=-0.916297857297 effort=33.5 velocity=28.6
- joint FR_hip_joint: limit lower=-0.802851455917 upper=0.802851455917 effort=33.5 velocity=21 -> lower=-0.802851455917 upper=0.802851455917 effort=33.5 velocity=52.4; origin xyz=0.1805 -0.047 0 rpy=0 0 0 -> xyz=0.183 -0.047 0 rpy=0 0 0
- joint FR_thigh_joint: limit lower=-1.0471975512 upper=4.18879020479 effort=33.5 velocity=21 -> lower=-1.0471975512 upper=4.18879020479 effort=33.5 velocity=28.6; origin xyz=0 -0.0838 0 rpy=0 0 0 -> xyz=0 -0.08505 0 rpy=0 0 0
- joint RL_calf_joint: limit lower=-2.69653369433 upper=-0.916297857297 effort=33.5 velocity=21 -> lower=-2.69653369433 upper=-0.916297857297 effort=33.5 velocity=28.6
- joint RL_hip_joint: limit lower=-0.802851455917 upper=0.802851455917 effort=33.5 velocity=21 -> lower=-0.802851455917 upper=0.802851455917 effort=33.5 velocity=52.4; origin xyz=-0.1805 0.047 0 rpy=0 0 0 -> xyz=-0.183 0.047 0 rpy=0 0 0
- joint RL_thigh_joint: limit lower=-1.0471975512 upper=4.18879020479 effort=33.5 velocity=21 -> lower=-1.0471975512 upper=4.18879020479 effort=33.5 velocity=28.6; origin xyz=0 0.0838 0 rpy=0 0 0 -> xyz=0 0.08505 0 rpy=0 0 0
- joint RR_calf_joint: limit lower=-2.69653369433 upper=-0.916297857297 effort=33.5 velocity=21 -> lower=-2.69653369433 upper=-0.916297857297 effort=33.5 velocity=28.6
- joint RR_hip_joint: limit lower=-0.802851455917 upper=0.802851455917 effort=33.5 velocity=21 -> lower=-0.802851455917 upper=0.802851455917 effort=33.5 velocity=52.4; origin xyz=-0.1805 -0.047 0 rpy=0 0 0 -> xyz=-0.183 -0.047 0 rpy=0 0 0
- joint RR_thigh_joint: limit lower=-1.0471975512 upper=4.18879020479 effort=33.5 velocity=21 -> lower=-1.0471975512 upper=4.18879020479 effort=33.5 velocity=28.6; origin xyz=0 -0.0838 0 rpy=0 0 0 -> xyz=0 -0.08505 0 rpy=0 0 0
