Commit message: add joint symmetry support for T1 head and torso

File: resources/robots/t1/urdf/T1_serial.urdf (robot description, URDF)
Before this commit: robot T1, 24 links, 23 joints
Links:
- link AL1: geometry visual mesh filename=../meshes/AL1.STL
- link AL2: geometry visual mesh filename=../meshes/AL2.STL
- link AL3: geometry collision cylinder length=0.15 radius=0.03; visual mesh filename=../meshes/AL3.STL
- link AR2: geometry visual mesh filename=../meshes/AR2.STL
- link AR3: geometry collision cylinder length=0.15 radius=0.03; visual mesh filename=../meshes/AR3.STL
- link Ankle_Cross_Left: geometry visual mesh filename=../meshes/Ankle_Cross_Left.STL
- link Ankle_Cross_Right: geometry visual mesh filename=../meshes/Ankle_Cross_Right.STL
- link H1: geometry visual mesh filename=../meshes/H1.STL
- link H2: geometry collision sphere radius=0.08; visual mesh filename=../meshes/H2.STL
- link Hip_Pitch_Left: geometry visual mesh filename=../meshes/Hip_Pitch_Left.STL
- link Hip_Pitch_Right: geometry visual mesh filename=../meshes/Hip_Pitch_Right.STL
- link Hip_Roll_Left: geometry visual mesh filename=../meshes/Hip_Roll_Left.STL
- link Hip_Roll_Right: geometry visual mesh filename=../meshes/Hip_Roll_Right.STL
- link Hip_Yaw_Left: geometry collision cylinder length=0.16 radius=0.05; visual mesh filename=../meshes/Hip_Yaw_Left.STL
- link Hip_Yaw_Right: geometry collision cylinder length=0.16 radius=0.05; visual mesh filename=../meshes/Hip_Yaw_Right.STL
- link Shank_Left: geometry collision cylinder length=0.15 radius=0.05; visual mesh filename=../meshes/Shank_Left.STL
- link Shank_Right: geometry collision cylinder length=0.15 radius=0.05; visual mesh filename=../meshes/Shank_Right.STL
- link Trunk: geometry collision box size=0.15 0.2 0.3; visual mesh filename=../meshes/Trunk.STL
- link Waist: geometry visual mesh filename=../meshes/Waist.STL
- link left_foot_link: geometry collision box size=0.223 0.1 0.03; visual mesh filename=../meshes/left_foot_link.STL
- link left_hand_link: geometry collision cylinder length=0.175 radius=0.03; visual mesh filename=../meshes/left_hand_link.STL
- link right_foot_link: geometry collision box size=0.223 0.1 0.03; visual mesh filename=../meshes/right_foot_link.STL
- link right_hand_link: geometry collision cylinder length=0.175 radius=0.03; visual mesh filename=../meshes/right_hand_link.STL

Commit message: fix T1 full body symmetry

File: resources/robots/t1/urdf/T1_serial.urdf (robot description, URDF)
Before this commit: robot T1, 24 links, 23 joints
Links:
- link AR1: geometry visual mesh filename=../meshes/AR1.STL

Commit message: add support for timm models

File: resources/robots/t1/urdf/T1_serial.urdf (robot description, URDF)
Before this commit: robot T1, 24 links, 23 joints
Joints:
- joint Left_Ankle_Pitch: limit lower=-0.87 upper=0.35 effort=20 velocity=18.8 -> lower=-0.87 upper=0.35 effort=24 velocity=18.8
- joint Left_Elbow_Yaw: origin xyz=0 0.1471 0 rpy=0 0 0 -> xyz=0 0.1471 0 rpy=0 0 -0.5
- joint Left_Hip_Roll: limit lower=-0.2 upper=1.57 effort=30 velocity=10.9 -> lower=-0.3 upper=1.57 effort=30 velocity=10.9
- joint Left_Shoulder_Pitch: origin xyz=0.0575 0.1063 0.219 rpy=0 0.00088113 0 -> xyz=0.0575 0.1063 0.219 rpy=0 0.2 0
- joint Left_Shoulder_Roll: origin xyz=0 0.047 0 rpy=0 0 0 -> xyz=0 0.047 0 rpy=-1.35 0 0
- joint Right_Ankle_Pitch: limit lower=-0.87 upper=0.35 effort=20 velocity=18.8 -> lower=-0.87 upper=0.35 effort=24 velocity=18.8
- joint Right_Elbow_Yaw: origin xyz=0 -0.1471 0 rpy=0 0 0 -> xyz=0 -0.1471 0 rpy=0 0 0.5
- joint Right_Hip_Roll: limit lower=-1.57 upper=0.2 effort=30 velocity=10.9 -> lower=-1.57 upper=0.3 effort=30 velocity=10.9
- joint Right_Shoulder_Pitch: origin xyz=0.0575 -0.1063 0.219 rpy=0 0.00088113 0 -> xyz=0.0575 -0.1063 0.219 rpy=0 0.2 0
- joint Right_Shoulder_Roll: origin xyz=0 -0.047 0 rpy=0 0 0 -> xyz=0 -0.047 0 rpy=1.35 0 0

Commit message: abring T1 config up to date

File: resources/robots/t1/urdf/T1_serial.urdf (robot description, URDF)
Before this commit: robot T1, 24 links, 23 joints
Joints:
- joint Left_Ankle_Pitch: limit lower=-0.87 upper=0.35 effort=24 velocity=18.8 -> lower=-0.87 upper=0.35 effort=20 velocity=18.8
- joint Left_Elbow_Yaw: origin xyz=0 0.1471 0 rpy=0 0 -0.5 -> xyz=0 0.1471 0 rpy=0 0 0
- joint Left_Hip_Roll: limit lower=-0.3 upper=1.57 effort=30 velocity=10.9 -> lower=-0.2 upper=1.57 effort=30 velocity=10.9
- joint Left_Shoulder_Pitch: origin xyz=0.0575 0.1063 0.219 rpy=0 0.2 0 -> xyz=0.0575 0.1063 0.219 rpy=0 0.00088113 0
- joint Left_Shoulder_Roll: origin xyz=0 0.047 0 rpy=-1.35 0 0 -> xyz=0 0.047 0 rpy=0 0 0
- joint Right_Ankle_Pitch: limit lower=-0.87 upper=0.35 effort=24 velocity=18.8 -> lower=-0.87 upper=0.35 effort=20 velocity=18.8
- joint Right_Elbow_Yaw: origin xyz=0 -0.1471 0 rpy=0 0 0.5 -> xyz=0 -0.1471 0 rpy=0 0 0
- joint Right_Hip_Roll: limit lower=-1.57 upper=0.3 effort=30 velocity=10.9 -> lower=-1.57 upper=0.2 effort=30 velocity=10.9
- joint Right_Shoulder_Pitch: origin xyz=0.0575 -0.1063 0.219 rpy=0 0.2 0 -> xyz=0.0575 -0.1063 0.219 rpy=0 0.00088113 0
- joint Right_Shoulder_Roll: origin xyz=0 -0.047 0 rpy=1.35 0 0 -> xyz=0 -0.047 0 rpy=0 0 0
